File: Codec.kicad_sch (KiCad schematic)
At the start: 28 parts, among them J2 PJ-316A-6A, U3 ES8327

Commit message: Did some things
Parts:
- C14, C18, C19: value 0.1uF -> 100nF
Changed lines of the file:
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@@
       (effects (font (size 1.27 1.27)) (justify right))
     )
-    (property "Value" "0.1uF" (at 153.67 53.34 0)
+    (property "Value" "100nF" (at 153.67 53.34 0)
       (effects (font (size 1.27 1.27)) (justify right))
     )
@@
       (effects (font (size 1.27 1.27)) (justify right))
     )
-    (property "Value" "0.1uF" (at 99.06 45.72 0)
+    (property "Value" "100nF" (at 99.06 45.72 0)
       (effects (font (size 1.27 1.27)) (justify right))
     )
@@
       (effects (font (size 1.27 1.27)) (justify right))
     )
-    (property "Value" "0.1uF" (at 140.97 43.18 0)
-      (effects (font (size 1.27 1.27)) (justify right))
-    )
+    (property "Value" "100nF" (at 140.97 43.18 0)
+      (effects (font (size 1.27 1.27)) (justify right))
+    )
