File: Music_32_V2.kicad_pcb (KiCad board)
At the start: 4 copper layers, 46 x 99.8 mm, 138 parts, among them J1 0.5-8P CTXJ-H2.0 119, J2 PJ-316A-6A, J3 U263-163N-4OS1735, J4 Micro_SD_Card_Det1, Q1 YJQ10N02A, Q2 YJQ10N02A, Q3 YJQD30P02A, Q4 YJQ10N02A, SW1 SEL, SW2 BOOT/HOME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

Commit message: Did some things
Parts:
- added C38: 100nF, Capacitor_SMD:C_0402_1005Metric, F.Cu at (132.4, 78.0)
- C1, C14, C18, C19, C2, C3, C4, C43, C5, C6, C7, C8, C9: value 0.1uF -> 100nF
Connections:
- BT1 pad 1: /Power/Batt+_unfuse -> Net-(Q1-D)
- BT1 pad 2: Net-(BT1--) -> /Power/Batt+_unfuse
- Q1 pad 3: Net-(BT1--) -> Net-(Q1-D)
- R33 pad 1: BATT+ -> /Power/Vin
Routing:
- net Net-(BT1--): track 17.6 -> 0.00 mm
- net Net-(Q1-D): track 0.00 -> 16.7 mm
- net BATT+: track 64.4 -> 50.6 mm
- net /Power/Vin: track 15.9 -> 23.7 mm
- net /Power/Batt+_unfuse: track 12.7 -> 19.9 mm
- net GND: track 159.0 -> 161.2 mm, vias 76 -> 77
- net +3.3V: track 254.4 -> 255.6 mm, vias 12 -> 13
Other:
- outline, holes or cut-outs redrawn
