File: Music_32_V2.kicad_sch (KiCad schematic)
At the start: 38 parts, among them J1 0.5-8P CTXJ-H2.0 119, SW1 SEL, SW2 BOOT/HOME, SW3 FF, SW4 RW, SW5 PP, SW6 RESET, U1 Sk-3393, U2 ESP32-S3-WROOM-1-N4R2

Commit message: Did some things
Parts:
- C1, C2, C3, C4, C5, C6, C7, C8, C9: value 0.1uF -> 100nF
Changed lines of the file:
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@@
   )
   (no_connect (at 74.93 92.71))
+  (bus_entry (at 115.57 62.23) (size 2.54 2.54)
+    (stroke (width 0) (type default))
+  )
   (wire (pts (xy 41.91 172.72) (xy 41.91 170.18))
     (stroke (width 0) (type default))
@@
       (effects (font (size 1.27 1.27)))
     )
-    (property "Value" "0.1uF" (at 123.19 176.53 90)
+    (property "Value" "100nF" (at 123.19 176.53 90)
       (effects (font (size 1.27 1.27)))
     )
@@
       (effects (font (size 1.27 1.27)))
     )
-    (property "Value" "0.1uF" (at 48.26 176.53 90)
+    (property "Value" "100nF" (at 48.26 176.53 90)
       (effects (font (size 1.27 1.27)))
     )
@@
       (effects (font (size 1.27 1.27)))
     )
-    (property "Value" "0.1uF" (at 71.12 102.87 0)
+    (property "Value" "100nF" (at 71.12 102.87 0)
       (effects (font (size 1.27 1.27)))
     )
@@
       (effects (font (size 1.27 1.27)))
     )
-    (property "Value" "0.1uF" (at 97.79 176.53 90)
+    (property "Value" "100nF" (at 97.79 176.53 90)
       (effects (font (size 1.27 1.27)))
     )
@@
       (effects (font (size 1.27 1.27)))
     )
-    (property "Value" "0.1uF" (at 73.66 176.53 90)
+    (property "Value" "100nF" (at 73.66 176.53 90)
       (effects (font (size 1.27 1.27)))
     )
@@
       (effects (font (size 1.27 1.27)))
     )
-    (property "Value" "0.1uF" (at 185.42 60.96 0)
+    (property "Value" "100nF" (at 185.42 60.96 0)
       (effects (font (size 1.27 1.27)))
     )
@@
       (effects (font (size 1.27 1.27)))
     )
-    (property "Value" "0.1uF" (at 55.88 102.87 0)
+    (property "Value" "100nF" (at 55.88 102.87 0)
       (effects (font (size 1.27 1.27)))
     )
@@
       (effects (font (size 1.27 1.27)))
     )
-    (property "Value" "0.1uF" (at 151.13 176.53 90)
+    (property "Value" "100nF" (at 151.13 176.53 90)
       (effects (font (size 1.27 1.27)))
     )
@@
   (symbol (lib_id "Device:C_Small") (at 238.76 57.15 0) (unit 1)
     (in_bom yes) (on_board yes) (dnp no) (fields_autoplaced)
-    (property "Reference" "C9" (at 241.3 55.8863 0)
+    (property "Reference" "C9" (at 241.3 56.5213 0)
       (effects (font (size 1.27 1.27)) (justify left))
     )
-    (property "Value" "0.1uF" (at 241.3 58.4263 0)
+    (property "Value" "100nF" (at 241.3 59.0613 0)
       (effects (font (size 1.27 1.27)) (justify left))
     )
