File: Peripherals.kicad_sch (KiCad schematic)
At the start: 23 parts, among them J4 Micro_SD_Card_Det1, Q4 YJQ10N02A, U10 PCF85063TP/1Z, U8 ST7889 2" LCD, U9 MAX17048, Y1 32.768KHz

Commit message: Did some things
Parts:
- added C38: 100nF, Capacitor_SMD:C_0402_1005Metric, symbol Device:C_Small
Connections:
- net +3.3V: now also C38.1
- net GND: now also C38.2
Changed lines of the file:
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@@
   (junction (at 180.34 110.49) (diameter 0) (color 0 0 0 0)
   )
+  (junction (at 172.72 134.62) (diameter 0) (color 0 0 0 0)
+  )
   (junction (at 54.61 39.37) (diameter 0) (color 0 0 0 0)
   )
@@
   )
   (junction (at 252.73 35.56) (diameter 0) (color 0 0 0 0)
+  )
+  (junction (at 167.64 107.95) (diameter 0) (color 0 0 0 0)
   )
   (junction (at 252.73 53.34) (diameter 0) (color 0 0 0 0)
@@
     (stroke (width 0) (type default))
   )
+  (wire (pts (xy 167.64 107.95) (xy 167.64 127))
+    (stroke (width 0) (type default))
+  )
+  (wire (pts (xy 167.64 107.95) (xy 194.31 107.95))
+    (stroke (width 0) (type default))
+  )
   (wire (pts (xy 54.61 39.37) (xy 59.69 39.37))
     (stroke (width 0) (type default))
@@
     (stroke (width 0) (type default))
   )
-  (wire (pts (xy 163.83 107.95) (xy 194.31 107.95))
+  (wire (pts (xy 163.83 107.95) (xy 167.64 107.95))
     (stroke (width 0) (type default))
   )
@@
     (stroke (width 0) (type default))
   )
+  (wire (pts (xy 172.72 134.62) (xy 167.64 134.62))
+    (stroke (width 0) (type default))
+  )
   (wire (pts (xy 158.75 44.45) (xy 167.64 44.45))
     (stroke (width 0) (type default))
@@
   )
   (wire (pts (xy 141.224 48.26) (xy 141.224 50.8))
+    (stroke (width 0) (type default))
+  )
+  (wire (pts (xy 167.64 134.62) (xy 167.64 132.08))
     (stroke (width 0) (type default))
   )
@@
     )
   )
+  (symbol (lib_id "Device:C_Small") (at 167.64 129.54 0) (unit 1)
+    (in_bom yes) (on_board yes) (dnp no)
+    (property "Reference" "C38" (at 161.798 128.778 0)
+      (effects (font (size 1.27 1.27)) (justify left))
+    )
+    (property "Value" "100nF" (at 160.02 130.81 0)
+      (effects (font (size 1.27 1.27)) (justify left))
+    )
+    (property "Footprint" "Capacitor_SMD:C_0402_1005Metric" (at 167.64 129.54 0)
+      (effects (font (size 1.27 1.27)) hide)
+    )
+    (property "Datasheet" "https://search.murata.co.jp/Ceramy/image/img/A01X/G101/ENG/GRT155C80J105KE01-01.pdf" (at 167.64 129.54 0)
+      (effects (font (size 1.27 1.27)) hide)
+    )
+    (property "DigiKeyLink" "https://www.digikey.ca/en/products/detail/murata-electronics/GRT155C80J105KE01J/13904934" (at 167.64 129.54 0)
+      (effects (font (size 1.27 1.27)) hide)
+    )
+    (property "Price" "0.0448" (at 167.64 129.54 0)
+      (effects (font (size 1.27 1.27)) hide)
+    )
+    (property "MPN" "490-GRT155C80J105KE01JCT-ND" (at 167.64 129.54 0)
+      (effects (font (size 1.27 1.27)) hide)
+    )
+    (property "MPN_LCSC" "C14445" (at 167.64 129.54 0)
+      (effects (font (size 1.27 1.27)) hide)
+    )
+    (property "Price_LCSC" "0.0018" (at 167.64 129.54 0)
+      (effects (font (size 1.27 1.27)) hide)
+    )
+    (property "LCSCLink" "https://lcsc.com/product-detail/Multilayer-Ceramic-Capacitors-MLCC-SMD-SMT_Samsung-Electro-Mechanics-CL05A105KP5NNNC_C14445.html" (at 167.64 129.54 0)
+      (effects (font (size 1.27 1.27)) hide)
+    )
+    (pin "1")
+    (pin "2")
+    (instances
+      (project "Music_32_V2"
+        (path "/14681cc8-ddd4-43ff-b571-daca84d76d6b/7e2784a5-f2e0-46a2-afdf-a2d608e4af43"
+          (reference "C38") (unit 1)
+        )
+      )
+      (project "Phone"
+        (path "/9a44bf40-ccf4-4ff9-bb89-c8bc2c0cf19f/08dec41e-a7ac-46dd-ad42-4ddeee026110/9e853077-f7a0-4acf-8837-d166e1e7fe64"
+          (reference "C?") (unit 1)
+        )
+      )
+      (project "Ipod"
+        (path "/c4cf9ad0-abea-4c32-bb0b-367e5261d002"
+          (reference "C?") (unit 1)
+        )
+        (path "/c4cf9ad0-abea-4c32-bb0b-367e5261d002/39f6bc4b-6dc6-4355-84d9-efa9a6355287"
+          (reference "C39") (unit 1)
+        )
+      )
+      (project "Power"
+        (path "/e4f8ce38-95ca-4021-bdd0-de4735b761e8"
+          (reference "C?") (unit 1)
+        )
+      )
+    )
+  )
   (symbol (lib_id "Device:R") (at 92.71 35.56 0) (mirror x) (unit 1)
     (in_bom yes) (on_board yes) (dnp no)
@@
   (symbol (lib_id "Diode:SZESD9B5.0ST5G") (at 172.72 130.81 90) (unit 1)
     (in_bom yes) (on_board yes) (dnp no)
-    (property "Reference" "D6" (at 170.18 130.175 90)
+    (property "Reference" "D6" (at 194.31 133.35 90)
       (effects (font (size 1.27 1.27)) (justify left))
     )
-    (property "Value" "SZESD9B5.0ST5G" (at 170.18 132.715 90)
+    (property "Value" "SZESD9B5.0ST5G" (at 200.66 137.16 90)
       (effects (font (size 1.27 1.27)) (justify left))
     )
